File: kicad-kria-4x-pmod.kicad_pcb (KiCad board)
At the start: 2 copper layers, 0 parts

Commit message: Initial commit
Parts:
- added C1: 100n, Capacitor_SMD:C_0603_1608Metric_Pad1.08x0.95mm_HandSolder, F.Cu at (100.3, 75.3)
- added C2: 100n, Capacitor_SMD:C_0603_1608Metric_Pad1.08x0.95mm_HandSolder, F.Cu at (135.5, 69.8)
- added C3: 100n, Capacitor_SMD:C_0603_1608Metric_Pad1.08x0.95mm_HandSolder, F.Cu at (158.3, 69.8)
- added H1: 2.5, MountingHole:MountingHole_2.5mm, F.Cu at (99.1, 81.9)
- added H2: 2.5, MountingHole:MountingHole_2.5mm, F.Cu at (129.5, 81.9)
- added H3: 2.5, MountingHole:MountingHole_2.5mm, F.Cu at (152.4, 81.9)
- added H4: 2.5, MountingHole:MountingHole_2.5mm, F.Cu at (106.7, 49.5)
- added H5: 2.5, MountingHole:MountingHole_2.5mm, F.Cu at (129.5, 49.5)
- added H6: 2.5, MountingHole:MountingHole_2.5mm, F.Cu at (152.4, 49.5)
- added J1: pmod-1, Library:PinHeader_2x06_P2.54mm_Horizontal, F.Cu at (101.6, 50.8)
- added J2: pmod-2, Library:PinHeader_2x06_P2.54mm_Horizontal, F.Cu at (124.5, 50.8)
- added J3: pmod-3, Library:PinHeader_2x06_P2.54mm_Horizontal, F.Cu at (147.3, 50.8)
- added J4: pmod-4, Library:PinHeader_2x06_P2.54mm_Horizontal, F.Cu at (170.2, 50.8)
- added J5: pmod-4 cable, Connector_IDC:IDC-Header_2x06_P2.54mm_Vertical, F.Cu at (167.6, 61.0)
- added J6: pmod 4, Connector_PinSocket_2.54mm:PinSocket_2x06_P2.54mm_Horizontal, F.Cu at (157.5, 73.7)
- added J7: pmod 3, Connector_PinSocket_2.54mm:PinSocket_2x06_P2.54mm_Horizontal, F.Cu at (134.6, 73.7)
- added J8: camera, Connector_PinSocket_2.54mm:PinSocket_2x09_P2.54mm_Horizontal, F.Cu at (104.1, 73.7)
Routing:
- net +3.3V: track 0.00 -> 176.5 mm
- net /h12: track 0.00 -> 30.7 mm
- net /d10: track 0.00 -> 30.7 mm
- net /e10: track 0.00 -> 30.7 mm
- net /c11: track 0.00 -> 30.7 mm
- net /e12: track 0.00 -> 30.7 mm
- net /d11: track 0.00 -> 30.7 mm
- net /b11: track 0.00 -> 30.7 mm
- net /b10: track 0.00 -> 30.7 mm
- net /ae10: track 0.00 -> 28.6 mm
- net /ad12: track 0.00 -> 28.6 mm
- net /af10: track 0.00 -> 28.6 mm
- net /ac12: track 0.00 -> 28.6 mm
- net /ad11: track 0.00 -> 28.5 mm
- net /aa11: track 0.00 -> 28.5 mm
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- added copper zone on B.Cu, net GND
- added copper zone on F.Cu, net GND
Other:
- board outline added: 91.4 x 41.9 mm
- board text added: "+3V3"
- board text added: "AA10"
- board text added: "AA11"
- board text added: "AC12"
- board text added: "AD10"
- board text added: "AD11"
- board text added: "AD12"
- board text added: "AE10"
- board text added: "AE12"
- board text added: "AF11"
- board text added: "AF12"
- board text added: "AG10"
- board text added: "AG11"
- board text added: "AH10"
- board text added: "AH11"
- board text added: "AH12"
- board text added: "B10"
- board text added: "B11"
- board text added: "C11"
- board text added: "D10"
- board text added: "D11"
- board text added: "E10"
- board text added: "E12"
- board text added: "F11"
- board text added: "F12"
- board text added: "G10"
- board text added: "GND"
- board text added: "H11"
- board text added: "H12"
- board text added: "J10"
- board text added: "J11"
- board text added: "K12"
- board text added: "K13"
- board text added: "kria-4x-pmod 1.0 2024-08-17 by S59MZ"
