File: kicad-kria-4x-pmod.kicad_sch (KiCad schematic)
At the start: 0 parts

Commit message: Initial commit
Parts:
- added C1, C2, C3: 100n, Capacitor_SMD:C_0603_1608Metric_Pad1.08x0.95mm_HandSolder, symbol Device:C
- added H1, H2, H3, H4, H5, H6: 2.5, MountingHole:MountingHole_2.5mm, symbol Mechanical:MountingHole
- added J1: pmod-1, Library:PinHeader_2x06_P2.54mm_Horizontal, symbol Connector_Generic:Conn_02x06_Odd_Even
- added J2: pmod-2, Library:PinHeader_2x06_P2.54mm_Horizontal, symbol Connector_Generic:Conn_02x06_Odd_Even
- added J3: pmod-3, Library:PinHeader_2x06_P2.54mm_Horizontal, symbol Connector_Generic:Conn_02x06_Odd_Even
- added J4: pmod-4, Library:PinHeader_2x06_P2.54mm_Horizontal, symbol Connector_Generic:Conn_02x06_Odd_Even
- added J5: pmod-4 cable, Connector_IDC:IDC-Header_2x06_P2.54mm_Vertical, symbol Connector_Generic:Conn_02x06_Odd_Even
- added J6: pmod 4, Connector_PinSocket_2.54mm:PinSocket_2x06_P2.54mm_Horizontal, symbol Connector_Generic:Conn_02x06_Odd_Even
- added J7: pmod 3, Connector_PinSocket_2.54mm:PinSocket_2x06_P2.54mm_Horizontal, symbol Connector_Generic:Conn_02x06_Odd_Even
- added J8: camera, Connector_PinSocket_2.54mm:PinSocket_2x09_P2.54mm_Horizontal, symbol Connector_Generic:Conn_02x09_Odd_Even
Connections:
- new net +3.3V: C1.1, C2.1, C3.1, J1.11 (Pin_11), J1.12 (Pin_12), J2.11 (Pin_11), J2.12 (Pin_12), J3.11 (Pin_11), J3.12 (Pin_12), J4.11 (Pin_11), J4.12 (Pin_12), J5.11 (Pin_11), J5.12 (Pin_12), J6.1 (Pin_1), J6.2 (Pin_2), J7.1 (Pin_1), J7.2 (Pin_2), J8.2 (Pin_2)
- new net GND: C1.2, C2.2, C3.2, J1.10 (Pin_10), J1.9 (Pin_9), J2.10 (Pin_10), J2.9 (Pin_9), J3.10 (Pin_10), J3.9 (Pin_9), J4.10 (Pin_10), J4.9 (Pin_9), J5.10 (Pin_10), J5.9 (Pin_9), J6.3 (Pin_3), J6.4 (Pin_4), J7.3 (Pin_3), J7.4 (Pin_4), J8.1 (Pin_1)
- new net aa10: J4.8 (Pin_8), J5.8 (Pin_8), J6.5 (Pin_5)
- new net aa11: J4.6 (Pin_6), J5.6 (Pin_6), J6.7 (Pin_7)
- new net ac12: J4.1 (Pin_1), J5.1 (Pin_1), J6.12 (Pin_12)
- new net ad10: J4.4 (Pin_4), J5.4 (Pin_4), J6.9 (Pin_9)
- new net ad11: J4.2 (Pin_2), J5.2 (Pin_2), J6.11 (Pin_11)
- new net ad12: J4.3 (Pin_3), J5.3 (Pin_3), J6.10 (Pin_10)
- new net ae10: J4.5 (Pin_5), J5.5 (Pin_5), J6.8 (Pin_8)
- new net ae12: J3.1 (Pin_1), J7.12 (Pin_12)
- new net af10: J4.7 (Pin_7), J5.7 (Pin_7), J6.6 (Pin_6)
- new net af11: J3.2 (Pin_2), J7.11 (Pin_11)
- new net af12: J3.3 (Pin_3), J7.10 (Pin_10)
- new net ag10: J3.5 (Pin_5), J7.8 (Pin_8)
- new net ag11: J3.4 (Pin_4), J7.9 (Pin_9)
- new net ah10: J3.7 (Pin_7), J7.6 (Pin_6)
- new net ah11: J3.8 (Pin_8), J7.5 (Pin_5)
- new net ah12: J3.6 (Pin_6), J7.7 (Pin_7)
- new net b10: J1.2 (Pin_2), J8.9 (Pin_9)
- new net b11: J1.8 (Pin_8), J8.3 (Pin_3)
- new net c11: J1.7 (Pin_7), J8.4 (Pin_4)
- new net d10: J1.5 (Pin_5), J8.6 (Pin_6)
- new net d11: J1.6 (Pin_6), J8.5 (Pin_5)
- new net e10: J1.3 (Pin_3), J8.8 (Pin_8)
- new net e12: J1.4 (Pin_4), J8.7 (Pin_7)
- new net f11: J2.8 (Pin_8), J8.11 (Pin_11)
- new net f12: J2.6 (Pin_6), J8.13 (Pin_13)
- new net g10: J2.4 (Pin_4), J8.15 (Pin_15)
- new net h11: J2.2 (Pin_2), J8.17 (Pin_17)
- new net h12: J1.1 (Pin_1), J8.10 (Pin_10)
- new net j10: J2.3 (Pin_3), J8.16 (Pin_16)
- new net j11: J2.1 (Pin_1), J8.18 (Pin_18)
- new net k12: J2.7 (Pin_7), J8.12 (Pin_12)
- new net k13: J2.5 (Pin_5), J8.14 (Pin_14)
